File: hardware/fencing1/left-side.kicad_sch (KiCad schematic)
At the start: 32 parts, among them SW3 SW_DPDT_x2, U3 NE555P, U4 LM324N_NOPB

Commit message: Working!
Parts:
- R29: value 1M -> 45K
Changed lines of the file:
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@@
       (effects (font (size 1.27 1.27)) (justify left))
     )
-    (property "Value" "1M" (at 269.24 124.46 0)
+    (property "Value" "45K" (at 269.24 124.46 0)
       (effects (font (size 1.27 1.27)) (justify left))
     )
