File: hardware/fencing1/right-side.kicad_sch (KiCad schematic)
At the start: 32 parts, among them SW1 SW_DPDT_x2, U5 NE555P, U6 LM324N_NOPB

Commit message: Working!
Parts:
- R44: value 1M -> 45K
Changed lines of the file:
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@@
       (effects (font (size 1.27 1.27)) (justify left))
     )
-    (property "Value" "1M" (at 270.51 124.46 0)
+    (property "Value" "45K" (at 270.51 124.46 0)
       (effects (font (size 1.27 1.27)) (justify left))
     )
